File: TRANSISTOR_LADDER_VCF_CORE_BC847BS.brd (EAGLE design)
At the start: 12.7 x 27.9 mm, 28 parts

Commit message: TRANSISTOR_LADDER_VCF_CORE
Parts:
- moved U$1 0.71 mm to (6.35, 25.4)
Routing:
- net C4A: track 19.3 -> 21.3 mm
- net V+: track 14.1 -> 15.2 mm
- net C3B: track 16.6 -> 17.4 mm
- net RL4: track 6.92 -> 7.69 mm
Other:
- board size 12.7 x 27.9 mm -> 12.7 x 29.2 mm
Changed lines of the file:
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@@
 <board>
 <plain>
-<wire x1="0" y1="25.66" x2="0" y2="-0.27" width="0" layer="20"/>
+<wire x1="0" y1="26.93" x2="0" y2="-0.27" width="0" layer="20"/>
 <wire x1="0" y1="-0.27" x2="1" y2="-1.27" width="0" layer="20" curve="90"/>
 <wire x1="1" y1="-1.27" x2="11.6875" y2="-1.27" width="0" layer="20"/>
 <wire x1="11.6875" y1="-1.27" x2="12.6875" y2="-0.27" width="0" layer="20" curve="90"/>
-<wire x1="12.6875" y1="-0.27" x2="12.6875" y2="25.66" width="0" layer="20"/>
-<wire x1="12.6875" y1="25.66" x2="11.6875" y2="26.66" width="0" layer="20" curve="90"/>
-<wire x1="11.6875" y1="26.66" x2="1" y2="26.66" width="0" layer="20"/>
-<wire x1="1" y1="26.66" x2="0" y2="25.66" width="0" layer="20" curve="90"/>
+<wire x1="12.6875" y1="-0.27" x2="12.6875" y2="26.93" width="0" layer="20"/>
+<wire x1="12.6875" y1="26.93" x2="11.6875" y2="27.93" width="0" layer="20" curve="90"/>
+<wire x1="11.6875" y1="27.93" x2="1" y2="27.93" width="0" layer="20"/>
+<wire x1="1" y1="27.93" x2="0" y2="26.93" width="0" layer="20" curve="90"/>
 <text x="3.175" y="25.4" size="0.8128" layer="25" rot="R45" align="center">V+</text>
 <text x="3.175" y="22.86" size="0.8128" layer="25" rot="R45" align="center">RL4</text>
@@
 <element name="V+" library="SparkFun-Connectors" package="1X01NS-KIT" value="M01NOSILK-KIT" x="1.27" y="25.4"/>
 <element name="RL4" library="SparkFun-Connectors" package="1X01NS-KIT" value="M01NOSILK-KIT" x="1.27" y="22.86"/>
-<element name="U$1" library="SparkFun-DiscreteSemi" package="SOT363" value="MMDT3904" x="6.0325" y="24.765" rot="R270"/>
+<element name="U$1" library="SparkFun-DiscreteSemi" package="SOT363" value="MMDT3904" x="6.35" y="25.4" rot="R270"/>
 <element name="U$2" library="SparkFun-DiscreteSemi" package="SOT363" value="MMDT3904" x="6.35" y="20.32" rot="R90"/>
 <element name="U$3" library="SparkFun-DiscreteSemi" package="SOT363" value="MMDT3904" x="6.35" y="15.24" rot="R270"/>
@@
 <contactref element="U$1" pad="3"/>
 <contactref element="U$1" pad="6"/>
-<wire x1="5.2325" y1="24.115" x2="5.55" y2="24.13" width="0.254" layer="1"/>
-<wire x1="5.55" y1="24.13" x2="5.715" y2="24.13" width="0.254" layer="1"/>
-<wire x1="5.715" y1="24.13" x2="5.715" y2="23.1775" width="0.254" layer="1"/>
-<via x="5.715" y="23.1775" extent="1-16" drill="0.5"/>
-<wire x1="5.715" y1="23.1775" x2="6.35" y2="23.8125" width="0.254" layer="16"/>
-<wire x1="6.35" y1="23.8125" x2="6.35" y2="25.0825" width="0.254" layer="16"/>
-<wire x1="6.35" y1="25.0825" x2="6.6675" y2="25.4" width="0.254" layer="16"/>
-<wire x1="6.6675" y1="25.4" x2="7.9375" y2="25.4" width="0.254" layer="16"/>
-<via x="7.9375" y="25.4" extent="1-16" drill="0.5"/>
-<wire x1="7.9375" y1="25.4" x2="6.985" y2="25.4" width="0.254" layer="1"/>
-<wire x1="6.985" y1="25.4" x2="6.985" y2="25.415" width="0.254" layer="1"/>
-<wire x1="6.985" y1="25.415" x2="6.8425" y2="25.415" width="0.254" layer="1"/>
+<wire x1="5.55" y1="24.75" x2="5.55" y2="24.765" width="0.254" layer="1"/>
+<wire x1="5.55" y1="24.765" x2="5.715" y2="24.765" width="0.254" layer="1"/>
+<wire x1="5.715" y1="24.765" x2="5.715" y2="24.13" width="0.254" layer="1"/>
+<via x="5.715" y="24.13" extent="1-16" drill="0.5"/>
+<wire x1="5.715" y1="24.13" x2="8.255" y2="26.67" width="0.254" layer="16"/>
+<via x="8.255" y="26.67" extent="1-16" drill="0.5"/>
+<wire x1="8.255" y1="26.67" x2="7.62" y2="26.035" width="0.254" layer="1"/>
+<wire x1="7.62" y1="26.035" x2="6.985" y2="26.035" width="0.254" layer="1"/>
+<wire x1="6.985" y1="26.035" x2="6.985" y2="26.05" width="0.254" layer="1"/>
+<wire x1="6.985" y1="26.05" x2="7.16" y2="26.05" width="0.254" layer="1"/>
 <wire x1="1.27" y1="25.4" x2="2.54" y2="25.4" width="0.254" layer="1"/>
-<wire x1="2.54" y1="25.4" x2="3.4925" y2="26.3525" width="0.254" layer="1"/>
-<wire x1="3.4925" y1="26.3525" x2="7.3025" y2="26.3525" width="0.254" layer="1"/>
-<wire x1="7.3025" y1="26.3525" x2="7.9375" y2="25.7175" width="0.254" layer="1"/>
-<wire x1="7.9375" y1="25.7175" x2="7.9375" y2="25.4" width="0.254" layer="1"/>
+<wire x1="2.54" y1="25.4" x2="3.175" y2="26.035" width="0.254" layer="1"/>
+<wire x1="3.175" y1="26.035" x2="3.175" y2="26.9875" width="0.254" layer="1"/>
+<wire x1="3.175" y1="26.9875" x2="3.81" y2="27.6225" width="0.254" layer="1"/>
+<wire x1="3.81" y1="27.6225" x2="7.62" y2="27.6225" width="0.254" layer="1"/>
+<wire x1="7.62" y1="27.6225" x2="8.255" y2="26.9875" width="0.254" layer="1"/>
+<wire x1="8.255" y1="26.9875" x2="8.255" y2="26.67" width="0.254" layer="1"/>
 </signal>
 <signal name="C2A">
@@
 <contactref element="U$1" pad="2"/>
 <contactref element="U$1" pad="5"/>
+<wire x1="5.55" y1="25.4" x2="7.16" y2="25.4" width="0.254" layer="1"/>
 <contactref element="RL4" pad="1"/>
-<wire x1="5.2325" y1="24.765" x2="6.8425" y2="24.765" width="0.254" layer="1"/>
-<wire x1="5.2325" y1="24.765" x2="4.7625" y2="24.765" width="0.254" layer="1"/>
-<wire x1="4.7625" y1="24.765" x2="4.445" y2="24.4475" width="0.254" layer="1"/>
-<wire x1="4.445" y1="24.4475" x2="4.445" y2="23.495" width="0.254" layer="1"/>
+<wire x1="5.55" y1="25.4" x2="5.08" y2="25.4" width="0.254" layer="1"/>
+<wire x1="5.08" y1="25.4" x2="4.445" y2="24.765" width="0.254" layer="1"/>
+<wire x1="4.445" y1="24.765" x2="4.445" y2="23.495" width="0.254" layer="1"/>
 <wire x1="4.445" y1="23.495" x2="3.81" y2="22.86" width="0.254" layer="1"/>
 <wire x1="3.81" y1="22.86" x2="1.27" y2="22.86" width="0.254" layer="1"/>
@@
 <contactref element="U$1" pad="4"/>
 <contactref element="U$2" pad="3"/>
-<wire x1="7.15" y1="24.115" x2="7.15" y2="20.97" width="0.254" layer="1"/>
+<wire x1="7.16" y1="24.75" x2="7.15" y2="24.75" width="0.254" layer="1"/>
+<wire x1="7.15" y1="24.75" x2="7.15" y2="20.97" width="0.254" layer="1"/>
 <contactref element="C4B" pad="1"/>
-<wire x1="6.8425" y1="24.115" x2="7.15" y2="24.115" width="0.254" layer="1"/>
-<wire x1="7.15" y1="24.115" x2="8.875" y2="24.115" width="0.254" layer="1"/>
-<wire x1="8.875" y1="24.115" x2="10.16" y2="25.4" width="0.254" layer="1"/>
+<wire x1="7.16" y1="24.75" x2="9.51" y2="24.75" width="0.254" layer="1"/>
+<wire x1="9.51" y1="24.75" x2="10.16" y2="25.4" width="0.254" layer="1"/>
 <wire x1="10.16" y1="25.4" x2="11.43" y2="25.4" width="0.254" layer="1"/>
 </signal>
@@
 <contactref element="U$2" pad="4"/>
 <wire x1="5.54" y1="20.97" x2="5.715" y2="20.97" width="0.254" layer="1"/>
-<wire x1="5.715" y1="20.97" x2="5.715" y2="21.9075" width="0.254" layer="1"/>
-<via x="5.715" y="21.9075" extent="1-16" drill="0.5"/>
-<wire x1="5.715" y1="21.9075" x2="5.715" y2="19.05" width="0.254" layer="16"/>
+<wire x1="5.715" y1="20.97" x2="5.715" y2="22.225" width="0.254" layer="1"/>
+<via x="5.715" y="22.225" extent="1-16" drill="0.5"/>
+<wire x1="5.715" y1="22.225" x2="5.715" y2="19.05" width="0.254" layer="16"/>
 <wire x1="5.715" y1="19.05" x2="5.08" y2="18.415" width="0.254" layer="16"/>
 <wire x1="5.08" y1="18.415" x2="5.715" y2="17.78" width="0.254" layer="16"/>
@@
 <wire x1="5.715" y1="14.425" x2="5.55" y2="14.59" width="0.254" layer="1"/>
 <contactref element="C3B" pad="1"/>
-<wire x1="11.43" y1="20.32" x2="9.8425" y2="20.32" width="0.254" layer="1"/>
-<wire x1="9.8425" y1="20.32" x2="8.255" y2="21.9075" width="0.254" layer="1"/>
-<via x="8.255" y="21.9075" extent="1-16" drill="0.5"/>
-<wire x1="8.255" y1="21.9075" x2="5.715" y2="21.9075" width="0.254" layer="16"/>
+<wire x1="11.43" y1="20.32" x2="10.16" y2="20.32" width="0.254" layer="1"/>
+<wire x1="10.16" y1="20.32" x2="8.255" y2="22.225" width="0.254" layer="1"/>
+<via x="8.255" y="22.225" extent="1-16" drill="0.5"/>
+<wire x1="8.255" y1="22.225" x2="5.715" y2="22.225" width="0.254" layer="16"/>
 </signal>
 <signal name="C4A">
 <contactref element="U$1" pad="1"/>
 <contactref element="U$2" pad="6"/>
-<wire x1="5.2325" y1="25.415" x2="4.43" y2="25.415" width="0.254" layer="1"/>
-<wire x1="4.43" y1="25.415" x2="4.445" y2="25.4" width="0.254" layer="1"/>
-<via x="4.445" y="25.4" extent="1-16" drill="0.5"/>
-<wire x1="4.445" y1="25.4" x2="4.445" y2="19.05" width="0.254" layer="16"/>
+<wire x1="5.55" y1="26.05" x2="5.065" y2="26.05" width="0.254" layer="1"/>
+<wire x1="5.065" y1="26.05" x2="4.445" y2="26.67" width="0.254" layer="1"/>
+<via x="4.445" y="26.67" extent="1-16" drill="0.5"/>
+<wire x1="4.445" y1="26.67" x2="4.445" y2="19.05" width="0.254" layer="16"/>
 <via x="4.445" y="19.05" extent="1-16" drill="0.5"/>
 <wire x1="4.445" y1="19.05" x2="5.065" y2="19.67" width="0.254" layer="1"/>
 <wire x1="5.065" y1="19.67" x2="5.54" y2="19.67" width="0.254" layer="1"/>
 <contactref element="C4A" pad="1"/>
-<wire x1="11.43" y1="22.86" x2="10.4775" y2="22.86" width="0.254" layer="1"/>
-<wire x1="10.4775" y1="22.86" x2="9.525" y2="21.9075" width="0.254" layer="1"/>
-<via x="9.525" y="21.9075" extent="1-16" drill="0.5"/>
-<wire x1="9.525" y1="21.9075" x2="9.525" y2="19.05" width="0.254" layer="16"/>
+<wire x1="11.43" y1="22.86" x2="10.16" y2="22.86" width="0.254" layer="1"/>
+<wire x1="10.16" y1="22.86" x2="9.525" y2="22.225" width="0.254" layer="1"/>
+<via x="9.525" y="22.225" extent="1-16" drill="0.5"/>
+<wire x1="9.525" y1="22.225" x2="9.525" y2="19.05" width="0.254" layer="16"/>
 <wire x1="9.525" y1="19.05" x2="8.89" y2="18.415" width="0.254" layer="16"/>
 <wire x1="8.89" y1="18.415" x2="6.35" y2="18.415" width="0.254" layer="16"/>
